File: kicad/bixi.kicad_pcb (KiCad board)
At the start: 2 copper layers, 87.5 x 100 mm, 40 parts, among them J1 RJ45, J10 Screw_Terminal_1x01, J2 RJ45, J3 RJ45, J4 RJ45, J5 RJ45, J6 RJ45, J7 RJ45, J8 RJ45, J9 Screw_Terminal_1x01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

Commit message: fix to silkscreen placement on bixi pcb
Parts:
- moved bm_streets 89.3 mm to (98.0, 143.0)
Changed lines of the file:
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@@
     (links 106)
     (no_connects 0)
-    (area 89.6582 -33.415001 185.152382 147.500001)
+    (area 90.085714 42.5 185.152382 149.368571)
     (thickness 1.6)
     (drawings 8)
@@
     (34 B.Paste user)
     (35 F.Paste user)
-    (36 B.SilkS user hide)
+    (36 B.SilkS user)
     (37 F.SilkS user)
     (38 B.Mask user)
@@
   )
   (module logos:bm_streets (layer F.Cu)
-    (at 91 54 90)
+    (at 98 143 90)
     (fp_text reference bm_streets (at 0 5 90) (layer B.SilkS) hide
       (effects (font (thickness 0.3)))
