File: kicad/bixi.sch (KiCad schematic (older format))
At the start: 34 parts, among them CON1 BARREL_JACK, J1 RJ45, J2 RJ45, J3 RJ45, J4 RJ45, J5 RJ45, J6 RJ45, J7 RJ45, J8 RJ45, U1 Teensy3.6, U2 SP3485CN, U3 SP3485CN, U4 SP3485CN, U5 SP3485CN, U6 SP3485CN, U7 SP3485CN, U8 SP3485CN, U9 SP3485CN

Commit message: kicad schematic and layout
Other:
- moved on the sheet: C1, C2, C3, C4, C5, C6, C7, C8, J1, J2, J3, J4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

Commit message: controller and receiver boards almost done for v1
Parts:
- C1, C2, C3, C4, C5, C6, C7, C8: footprint Capacitors_THT:C_Disc_D3.0mm_W1.6mm_P2.50mm -> Capacitors_THT:C_Disc_D3_P2.5
- R1, R2, R3, R4, R5, R6, R7, R8: footprint Resistors_THT:R_Axial_DIN0207_L6.3mm_D2.5mm_P7.62mm_Horizontal -> Resistors_THT:Resistor_Horizontal_RM7mm
Changed lines of the file:
@@
 F 0 "R8" V 9180 5450 50  0000 C CNN
 F 1 "100" V 9100 5450 50  0000 C CNN
-F 2 "Resistors_THT:R_Axial_DIN0207_L6.3mm_D2.5mm_P7.62mm_Horizontal" V 9030 5450 50  0001 C CNN
+F 2 "Resistors_THT:Resistor_Horizontal_RM7mm" V 9030 5450 50  0001 C CNN
 F 3 "" H 9100 5450 50  0000 C CNN
 	1    9100 5450
@@
 F 0 "R7" V 9180 4200 50  0000 C CNN
 F 1 "100" V 9100 4200 50  0000 C CNN
-F 2 "Resistors_THT:R_Axial_DIN0207_L6.3mm_D2.5mm_P7.62mm_Horizontal" V 9030 4200 50  0001 C CNN
+F 2 "Resistors_THT:Resistor_Horizontal_RM7mm" V 9030 4200 50  0001 C CNN
 F 3 "" H 9100 4200 50  0000 C CNN
 	1    9100 4200
@@
 F 0 "R6" V 9180 2950 50  0000 C CNN
 F 1 "100" V 9100 2950 50  0000 C CNN
-F 2 "Resistors_THT:R_Axial_DIN0207_L6.3mm_D2.5mm_P7.62mm_Horizontal" V 9030 2950 50  0001 C CNN
+F 2 "Resistors_THT:Resistor_Horizontal_RM7mm" V 9030 2950 50  0001 C CNN
 F 3 "" H 9100 2950 50  0000 C CNN
 	1    9100 2950
@@
 F 0 "R5" V 9180 1700 50  0000 C CNN
 F 1 "100" V 9100 1700 50  0000 C CNN
-F 2 "Resistors_THT:R_Axial_DIN0207_L6.3mm_D2.5mm_P7.62mm_Horizontal" V 9030 1700 50  0001 C CNN
+F 2 "Resistors_THT:Resistor_Horizontal_RM7mm" V 9030 1700 50  0001 C CNN
 F 3 "" H 9100 1700 50  0000 C CNN
 	1    9100 1700
@@
 F 0 "R4" V 6380 5550 50  0000 C CNN
 F 1 "100" V 6300 5550 50  0000 C CNN
-F 2 "Resistors_THT:R_Axial_DIN0207_L6.3mm_D2.5mm_P7.62mm_Horizontal" V 6230 5550 50  0001 C CNN
+F 2 "Resistors_THT:Resistor_Horizontal_RM7mm" V 6230 5550 50  0001 C CNN
 F 3 "" H 6300 5550 50  0000 C CNN
 	1    6300 5550
@@
 F 0 "R3" V 6380 4300 50  0000 C CNN
 F 1 "100" V 6300 4300 50  0000 C CNN
-F 2 "Resistors_THT:R_Axial_DIN0207_L6.3mm_D2.5mm_P7.62mm_Horizontal" V 6230 4300 50  0001 C CNN
+F 2 "Resistors_THT:Resistor_Horizontal_RM7mm" V 6230 4300 50  0001 C CNN
 F 3 "" H 6300 4300 50  0000 C CNN
 	1    6300 4300
@@
 F 0 "R2" V 6380 3050 50  0000 C CNN
 F 1 "100" V 6300 3050 50  0000 C CNN
-F 2 "Resistors_THT:R_Axial_DIN0207_L6.3mm_D2.5mm_P7.62mm_Horizontal" V 6230 3050 50  0001 C CNN
+F 2 "Resistors_THT:Resistor_Horizontal_RM7mm" V 6230 3050 50  0001 C CNN
 F 3 "" H 6300 3050 50  0000 C CNN
 	1    6300 3050
@@
 F 0 "R1" V 6380 1800 50  0000 C CNN
 F 1 "100" V 6300 1800 50  0000 C CNN
-F 2 "Resistors_THT:R_Axial_DIN0207_L6.3mm_D2.5mm_P7.62mm_Horizontal" V 6230 1800 50  0001 C CNN
+F 2 "Resistors_THT:Resistor_Horizontal_RM7mm" V 6230 1800 50  0001 C CNN
 F 3 "" H 6300 1800 50  0000 C CNN
 	1    6300 1800
@@
 F 0 "C1" H 4325 6400 50  0000 L CNN
 F 1 "C" H 4325 6200 50  0000 L CNN
-F 2 "Capacitors_THT:C_Disc_D3.0mm_W1.6mm_P2.50mm" H 4338 6150 50  0001 C CNN
+F 2 "Capacitors_THT:C_Disc_D3_P2.5" H 4338 6150 50  0001 C CNN
 F 3 "" H 4300 6300 50  0000 C CNN
 	1    4300 6300
@@
 F 0 "C2" H 4525 6400 50  0000 L CNN
 F 1 "C" H 4525 6200 50  0000 L CNN
-F 2 "Capacitors_THT:C_Disc_D3.0mm_W1.6mm_P2.50mm" H 4538 6150 50  0001 C CNN
+F 2 "Capacitors_THT:C_Disc_D3_P2.5" H 4538 6150 50  0001 C CNN
 F 3 "" H 4500 6300 50  0000 C CNN
 	1    4500 6300
@@
 F 0 "C3" H 4725 6400 50  0000 L CNN
 F 1 "C" H 4725 6200 50  0000 L CNN
-F 2 "Capacitors_THT:C_Disc_D3.0mm_W1.6mm_P2.50mm" H 4738 6150 50  0001 C CNN
+F 2 "Capacitors_THT:C_Disc_D3_P2.5" H 4738 6150 50  0001 C CNN
 F 3 "" H 4700 6300 50  0000 C CNN
 	1    4700 6300
@@
 F 0 "C4" H 4925 6400 50  0000 L CNN
 F 1 "C" H 4925 6200 50  0000 L CNN
-F 2 "Capacitors_THT:C_Disc_D3.0mm_W1.6mm_P2.50mm" H 4938 6150 50  0001 C CNN
+F 2 "Capacitors_THT:C_Disc_D3_P2.5" H 4938 6150 50  0001 C CNN
 F 3 "" H 4900 6300 50  0000 C CNN
 	1    4900 6300
@@
 F 0 "C5" H 5125 6400 50  0000 L CNN
 F 1 "C" H 5125 6200 50  0000 L CNN
-F 2 "Capacitors_THT:C_Disc_D3.0mm_W1.6mm_P2.50mm" H 5138 6150 50  0001 C CNN
+F 2 "Capacitors_THT:C_Disc_D3_P2.5" H 5138 6150 50  0001 C CNN
 F 3 "" H 5100 6300 50  0000 C CNN
 	1    5100 6300
@@
 F 0 "C6" H 5325 6400 50  0000 L CNN
 F 1 "C" H 5325 6200 50  0000 L CNN
-F 2 "Capacitors_THT:C_Disc_D3.0mm_W1.6mm_P2.50mm" H 5338 6150 50  0001 C CNN
+F 2 "Capacitors_THT:C_Disc_D3_P2.5" H 5338 6150 50  0001 C CNN
 F 3 "" H 5300 6300 50  0000 C CNN
 	1    5300 6300
@@
 F 0 "C7" H 5525 6400 50  0000 L CNN
 F 1 "C" H 5525 6200 50  0000 L CNN
-F 2 "Capacitors_THT:C_Disc_D3.0mm_W1.6mm_P2.50mm" H 5538 6150 50  0001 C CNN
+F 2 "Capacitors_THT:C_Disc_D3_P2.5" H 5538 6150 50  0001 C CNN
 F 3 "" H 5500 6300 50  0000 C CNN
 	1    5500 6300
@@
 F 0 "C8" H 5725 6400 50  0000 L CNN
 F 1 "C" H 5725 6200 50  0000 L CNN
-F 2 "Capacitors_THT:C_Disc_D3.0mm_W1.6mm_P2.50mm" H 5738 6150 50  0001 C CNN
+F 2 "Capacitors_THT:C_Disc_D3_P2.5" H 5738 6150 50  0001 C CNN
 F 3 "" H 5700 6300 50  0000 C CNN
 	1    5700 6300

Commit message: controller board screw terminal, screw holes. ready for build
Parts:
- removed CON1: BARREL_JACK, Connectors:BARREL_JACK, symbol BARREL_JACK
- added J9: Screw_Terminal_1x02, custom:HB9500-2P, symbol Screw_Terminal_1x02
Connections:
- no-connect marks 9 -> 8
Changed lines of the file:
@@
 WS_8
-$Comp
-L BARREL_JACK CON1
-U 1 1 58BF152F
-P 3450 6050
-F 0 "CON1" H 3450 6300 50  0000 C CNN
-F 1 "BARREL_JACK" H 3450 5850 50  0000 C CNN
-F 2 "Connectors:BARREL_JACK" H 3450 6050 50  0001 C CNN
-F 3 "" H 3450 6050 50  0000 C CNN
-	1    3450 6050
-	1    0    0    -1
-$EndComp
 $Comp
 L GND #PWR057
@@
 	1    0    0    -1
 $EndComp
-NoConn ~ 3750 6050
 $Comp
 L C C1
@@
 Connection ~ 6150 4300
 Connection ~ 6150 5550
+$Comp
+L Screw_Terminal_1x02 J9
+U 1 1 58E14E9C
+P 3550 6050
+F 0 "J9" H 3550 6300 50  0000 C TNN
+F 1 "Screw_Terminal_1x02" V 3400 6050 50  0000 C TNN
+F 2 "custom:HB9500-2P" H 3550 5825 50  0001 C CNN
+F 3 "" H 3525 6050 50  0001 C CNN
+	1    3550 6050
+	1    0    0    -1
+$EndComp
 $EndSCHEMATC

Commit message: both pcb's sent to fab
Parts:
- removed J9: Screw_Terminal_1x02, custom:HB9500-2P, symbol Screw_Terminal_1x02
- added J10, J9: Screw_Terminal_1x01, custom:A116169CT_SPADE_CONNECTOR, symbol Screw_Terminal_1x01
Changed lines of the file:
@@
 LIBS:valves
 LIBS:teensy
-LIBS:bixi-cache
 EELAYER 25 0
 EELAYER END
@@
 L GND #PWR057
 U 1 1 58BF15B9
-P 3750 6150
-F 0 "#PWR057" H 3750 5900 50  0001 C CNN
-F 1 "GND" H 3750 6000 50  0000 C CNN
-F 2 "" H 3750 6150 50  0000 C CNN
-F 3 "" H 3750 6150 50  0000 C CNN
-	1    3750 6150
+P 3750 6300
+F 0 "#PWR057" H 3750 6050 50  0001 C CNN
+F 1 "GND" H 3750 6150 50  0000 C CNN
+F 2 "" H 3750 6300 50  0000 C CNN
+F 3 "" H 3750 6300 50  0000 C CNN
+	1    3750 6300
 	1    0    0    -1
 $EndComp
@@
 $EndComp
 Wire Wire Line
-	5700 6150 4300 6150
+	4300 6150 5700 6150
 Wire Wire Line
 	4300 6450 5700 6450
@@
 Connection ~ 6150 5550
 $Comp
-L Screw_Terminal_1x02 J9
-U 1 1 58E14E9C
-P 3550 6050
-F 0 "J9" H 3550 6300 50  0000 C TNN
-F 1 "Screw_Terminal_1x02" V 3400 6050 50  0000 C TNN
-F 2 "custom:HB9500-2P" H 3550 5825 50  0001 C CNN
-F 3 "" H 3525 6050 50  0001 C CNN
-	1    3550 6050
-	1    0    0    -1
-$EndComp
+L Screw_Terminal_1x01 J9
+U 1 1 58EA496D
+P 3550 5950
+F 0 "J9" H 3550 6100 50  0000 C TNN
+F 1 "Screw_Terminal_1x01" V 3400 5950 50  0000 C TNN
+F 2 "custom:A116169CT_SPADE_CONNECTOR" H 3550 5825 50  0001 C CNN
+F 3 "" H 3550 5850 50  0001 C CNN
+	1    3550 5950
+	1    0    0    -1
+$EndComp
+$Comp
+L Screw_Terminal_1x01 J10
+U 1 1 58EA4A14
+P 3550 6300
+F 0 "J10" H 3550 6450 50  0000 C TNN
+F 1 "Screw_Terminal_1x01" V 3400 6300 50  0000 C TNN
+F 2 "custom:A116169CT_SPADE_CONNECTOR" H 3550 6175 50  0001 C CNN
+F 3 "" H 3550 6200 50  0001 C CNN
+	1    3550 6300
+	1    0    0    -1
+$EndComp

Commit message: bixi node updates
Parts:
- removed J10, J9: Screw_Terminal_1x01, custom:A116169CT_SPADE_CONNECTOR, symbol Screw_Terminal_1x01
Changed lines of the file:
@@
 LIBS:valves
 LIBS:teensy
+LIBS:bixi-cache
 EELAYER 25 0
 EELAYER END
@@
 WS_8
 $Comp
-L GND #PWR057
-U 1 1 58BF15B9
-P 3750 6300
-F 0 "#PWR057" H 3750 6050 50  0001 C CNN
-F 1 "GND" H 3750 6150 50  0000 C CNN
-F 2 "" H 3750 6300 50  0000 C CNN
-F 3 "" H 3750 6300 50  0000 C CNN
-	1    3750 6300
-	1    0    0    -1
-$EndComp
-$Comp
-L VCC #PWR058
-U 1 1 58BF164F
-P 3750 5950
-F 0 "#PWR058" H 3750 5800 50  0001 C CNN
-F 1 "VCC" H 3750 6100 50  0000 C CNN
-F 2 "" H 3750 5950 50  0000 C CNN
-F 3 "" H 3750 5950 50  0000 C CNN
-	1    3750 5950
-	1    0    0    -1
-$EndComp
-$Comp
 L C C1
 U 1 1 58BF16CF
@@
 Connection ~ 6150 4300
 Connection ~ 6150 5550
-$Comp
-L Screw_Terminal_1x01 J9
-U 1 1 58EA496D
-P 3550 5950
-F 0 "J9" H 3550 6100 50  0000 C TNN
-F 1 "Screw_Terminal_1x01" V 3400 5950 50  0000 C TNN
-F 2 "custom:A116169CT_SPADE_CONNECTOR" H 3550 5825 50  0001 C CNN
-F 3 "" H 3550 5850 50  0001 C CNN
-	1    3550 5950
-	1    0    0    -1
-$EndComp
-$Comp
-L Screw_Terminal_1x01 J10
-U 1 1 58EA4A14
-P 3550 6300
-F 0 "J10" H 3550 6450 50  0000 C TNN
-F 1 "Screw_Terminal_1x01" V 3400 6300 50  0000 C TNN
-F 2 "custom:A116169CT_SPADE_CONNECTOR" H 3550 6175 50  0001 C CNN
-F 3 "" H 3550 6200 50  0001 C CNN
-	1    3550 6300
-	1    0    0    -1
-$EndComp
 $EndSCHEMATC

Commit message: v3 pcb first pass
Parts:
- removed C2, C3, C4, C5, C6, C7, C8: C, Capacitors_THT:C_Disc_D3_P2.5, symbol C
- removed U2, U3, U4, U5, U6, U7, U8, U9: SP3485CN, Housings_DIP:DIP-8_W7.62mm, symbol SP3485CN
- added U2: sn75lbc978, Housings_SSOP:SSOP-56_7.5x18.5mm_Pitch0.635mm, symbol sn75lbc978
- added U3: ESP8266, custom:ESP8266, symbol ESP8266
- C1: footprint Capacitors_THT:C_Disc_D3_P2.5 -> Capacitors_THT:C_Disc_D4.7mm_W2.5mm_P5.00mm
- R1, R2, R3, R4, R5, R6, R7, R8: footprint Resistors_THT:Resistor_Horizontal_RM7mm -> Resistors_THT:R_Axial_DIN0207_L6.3mm_D2.5mm_P7.62mm_Horizontal
Connections:
- net GND: now also U2.13 (GND), U2.14 (GND), U2.15 (GND), U2.16 (GND), U2.17 (GND), U2.2 (WRAP2), U2.3 (WRAP1), U2.40 (GND), U2.41 (GND), U2.42 (GND), U2.43 (GND), U2.44 (GND), U3.1 (GND); no longer J1.9 (SHIELD), J2.9 (SHIELD), J3.9 (SHIELD), J4.9 (SHIELD), J5.9 (SHIELD), J6.9 (SHIELD), J7.9 (SHIELD), J8.9 (SHIELD)
- net VCC: now also U2.11 (4DE/~RE), U2.12 (VCC), U2.18 (VCC), U2.20 (5DE/~RE), U2.22 (6DE/~RE), U2.24 (7DE/~RE), U2.26 (8DE/~RE), U2.39 (VCC), U2.45 (VCC), U2.5 (1DE/~RE), U2.54 (CE), U2.7 (2DE/~RE), U2.9 (3DE/~RE)
- net WS_1: now also U2.4 (1A)
- net WS_2: now also U2.6 (2A)
- net WS_3: now also U2.8 (3A)
- net WS_4: now also U2.10 (4A)
- net WS_5: now also U2.19 (5A)
- net WS_6: now also U2.21 (6A)
- net WS_7: now also U2.23 (7A)
- net WS_8: now also U2.25 (8A)
- net 8A: now reaches J8.1
- net 8A: now also R8.2, U2.51 (8B+); no longer R8.1
- net 8B: now reaches J8.2
- net 8B: now also R8.1, U2.50 (8B-); no longer R8.2
- net 3V: now reaches U1.75 (3.3V)
- net 3V: now also U3.8 (3V)
- net 7A: now reaches J7.1
- net 7A: now also R7.2, U2.49 (7B+); no longer R7.1
- net 7B: now reaches J7.2
- net 7B: now also R7.1, U2.48 (7B-); no longer R7.2
- net 6A: now reaches J6.1
- net 6A: now also R6.2, U2.47 (6B+); no longer R6.1
- net 6B: now reaches J6.2
- net 6B: now also R6.1, U2.46 (6B-); no longer R6.2
- net 5A: now reaches J5.1
- net 5A: now also R5.2, U2.38 (5B+); no longer R5.1
- net 5B: now reaches J5.2
- net 5B: now also R5.1, U2.37 (5B-); no longer R5.2
- net 4A: now reaches J4.1
- net 4A: now also R4.2, U2.36 (4B+); no longer R4.1
- net 4B: now reaches J4.2
- net 4B: now also R4.1, U2.35 (4B-); no longer R4.2
- net 3A: now reaches J3.1
- net 3A: now also R3.2, U2.34 (3B+); no longer R3.1
- net 3B: now reaches J3.2
- net 3B: now also R3.1, U2.33 (3B-); no longer R3.2
- net 2A: now reaches J2.1
- net 2A: now also R2.2, U2.32 (2B+); no longer R2.1
- net 2B: now reaches J2.2
- net 2B: now also R2.1, U2.31 (2B-); no longer R2.2
- net 1A: now reaches J1.1
- net 1A: now also R1.2, U2.30 (1B+); no longer R1.1
- net 1B: now reaches J1.2
- net 1B: now also R1.1, U2.29 (1B-); no longer R1.2
- no-connect marks 8 -> 6
Other:
- moved on the sheet: C1, J1, J2, J3, J4, J5, J6, J7, J8
