File: kicad/bixi_pt/bixi_pt.sch (KiCad schematic (older format))
At the start: 3 parts, among them J1 Screw_Terminal_1x02, J2 CONN_01X03, J3 CONN_01X03

Commit message: v3 pcb's plotted, ready for fab
Parts:
- J2, J3: footprint Connectors_JST:JST_XH_B03B-XH-A_03x2.50mm_Straight -> custom:PAD_3X_OVAL_WS2812B
Changed lines of the file:
@@
 LIBS:contrib
 LIBS:valves
+LIBS:bixi_pt-cache
 EELAYER 25 0
 EELAYER END
@@
 F 0 "J2" H 4500 3050 50  0000 C CNN
 F 1 "CONN_01X03" V 4600 2850 50  0000 C CNN
-F 2 "Connectors_JST:JST_XH_B03B-XH-A_03x2.50mm_Straight" H 4500 2850 50  0001 C CNN
+F 2 "custom:PAD_3X_OVAL_WS2812B" H 4500 2850 50  0001 C CNN
 F 3 "" H 4500 2850 50  0001 C CNN
 	1    4500 2850
@@
 F 0 "J3" H 6800 3050 50  0000 C CNN
 F 1 "CONN_01X03" V 6900 2850 50  0000 C CNN
-F 2 "Connectors_JST:JST_XH_B03B-XH-A_03x2.50mm_Straight" H 6800 2850 50  0001 C CNN
+F 2 "custom:PAD_3X_OVAL_WS2812B" H 6800 2850 50  0001 C CNN
 F 3 "" H 6800 2850 50  0001 C CNN
 	1    6800 2850

Commit message: first changes for v4 pcb's
Parts:
- added PWR_L1, PWR_R1: Jumper, Pin_Headers:Pin_Header_Straight_1x02_Pitch2.54mm, symbol Jumper
- renumbered J2 to L1, J3 to R1
Connections:
- net VCC: now also PWR_L1.2, PWR_R1.1; no longer L1.3 (P3), R1.1 (P1)
- new net VCCL: L1.3 (P3), PWR_L1.1
- new net VCCR: PWR_R1.2, R1.1 (P1)
Changed lines of the file:
@@
 GND
 $Comp
-L CONN_01X03 J2
+L CONN_01X03 L1
 U 1 1 5907F1DC
 P 4500 2850
-F 0 "J2" H 4500 3050 50  0000 C CNN
+F 0 "L1" H 4500 3050 50  0000 C CNN
 F 1 "CONN_01X03" V 4600 2850 50  0000 C CNN
 F 2 "custom:PAD_3X_OVAL_WS2812B" H 4500 2850 50  0001 C CNN
@@
 Text Label 4300 2750 2    60   ~ 0
 GND
-Text Label 4300 2950 2    60   ~ 0
-VCC
 Text Label 4300 2850 2    60   ~ 0
 DATA
 $Comp
-L CONN_01X03 J3
+L CONN_01X03 R1
 U 1 1 5907F236
 P 6800 2850
-F 0 "J3" H 6800 3050 50  0000 C CNN
+F 0 "R1" H 6800 3050 50  0000 C CNN
 F 1 "CONN_01X03" V 6900 2850 50  0000 C CNN
 F 2 "custom:PAD_3X_OVAL_WS2812B" H 6800 2850 50  0001 C CNN
@@
 Text Label 7000 2850 0    60   ~ 0
 DATA
+$Comp
+L Jumper PWR_L1
+U 1 1 59139D88
+P 5550 3550
+F 0 "PWR_L1" H 5550 3700 50  0000 C CNN
+F 1 "Jumper" H 5550 3470 50  0000 C CNN
+F 2 "Pin_Headers:Pin_Header_Straight_1x02_Pitch2.54mm" H 5550 3550 50  0001 C CNN
+F 3 "" H 5550 3550 50  0001 C CNN
+	1    5550 3550
+	1    0    0    -1
+$EndComp
+Text Label 4300 2950 2    60   ~ 0
+VCCL
 Text Label 7000 2950 0    60   ~ 0
+VCCR
+Text Label 5250 3550 2    60   ~ 0
+VCCL
+Text Label 5850 3550 0    60   ~ 0
 VCC
+$Comp
+L Jumper PWR_R1
+U 1 1 59139ED6
+P 5550 3900
+F 0 "PWR_R1" H 5550 4050 50  0000 C CNN
+F 1 "Jumper" H 5550 3820 50  0000 C CNN
+F 2 "Pin_Headers:Pin_Header_Straight_1x02_Pitch2.54mm" H 5550 3900 50  0001 C CNN
+F 3 "" H 5550 3900 50  0001 C CNN
+	1    5550 3900
+	1    0    0    -1
+$EndComp
+Text Label 5250 3900 2    60   ~ 0
+VCC
+Text Label 5850 3900 0    60   ~ 0
+VCCR
 $EndSCHEMATC

Commit message: new power injection board is ready
Parts:
- J1: footprint custom:HP_9500_Terminal_Connector -> custom:OSTYK42102030-2P-Terminal
- L1, R1: footprint custom:PAD_3X_OVAL_WS2812B -> custom:3-wire-hole-with-relief
Connections:
- net GND: now also L1.3 (P3), R1.1 (P1); no longer L1.1 (P1), R1.3 (P3)
- net VCCL: now also L1.1 (P1); no longer L1.3 (P3)
- net VCCR: now also R1.3 (P3); no longer R1.1 (P1)
Other:
- moved on the sheet: J1
Changed lines of the file:
@@
 L Screw_Terminal_1x02 J1
 U 1 1 5907F10E
-P 5550 2850
-F 0 "J1" H 5550 3100 50  0000 C TNN
-F 1 "Screw_Terminal_1x02" V 5400 2850 50  0000 C TNN
-F 2 "custom:HP_9500_Terminal_Connector" H 5550 2625 50  0001 C CNN
-F 3 "" H 5525 2850 50  0001 C CNN
-	1    5550 2850
+P 6000 2850
+F 0 "J1" H 6000 3100 50  0000 C TNN
+F 1 "Screw_Terminal_1x02" V 5850 2850 50  0000 C TNN
+F 2 "custom:OSTYK42102030-2P-Terminal" H 6000 2625 50  0001 C CNN
+F 3 "" H 5975 2850 50  0001 C CNN
+	1    6000 2850
 	1    0    0    -1
 $EndComp
-Text Label 5750 2750 0    60   ~ 0
+Text Label 6200 2750 0    60   ~ 0
 VCC
-Text Label 5750 2950 0    60   ~ 0
+Text Label 6200 2950 0    60   ~ 0
 GND
 $Comp
@@
 F 0 "L1" H 4500 3050 50  0000 C CNN
 F 1 "CONN_01X03" V 4600 2850 50  0000 C CNN
-F 2 "custom:PAD_3X_OVAL_WS2812B" H 4500 2850 50  0001 C CNN
+F 2 "custom:3-wire-hole-with-relief" H 4500 2850 50  0001 C CNN
 F 3 "" H 4500 2850 50  0001 C CNN
 	1    4500 2850
 	1    0    0    -1
 $EndComp
-Text Label 4300 2750 2    60   ~ 0
+Text Label 4300 2950 2    60   ~ 0
 GND
 Text Label 4300 2850 2    60   ~ 0
@@
 F 0 "R1" H 6800 3050 50  0000 C CNN
 F 1 "CONN_01X03" V 6900 2850 50  0000 C CNN
-F 2 "custom:PAD_3X_OVAL_WS2812B" H 6800 2850 50  0001 C CNN
+F 2 "custom:3-wire-hole-with-relief" H 6800 2850 50  0001 C CNN
 F 3 "" H 6800 2850 50  0001 C CNN
 	1    6800 2850
 	-1   0    0    1
 $EndComp
-Text Label 7000 2750 0    60   ~ 0
+Text Label 7000 2950 0    60   ~ 0
 GND
 Text Label 7000 2850 0    60   ~ 0
@@
 	1    0    0    -1
 $EndComp
-Text Label 4300 2950 2    60   ~ 0
+Text Label 4300 2750 2    60   ~ 0
 VCCL
-Text Label 7000 2950 0    60   ~ 0
+Text Label 7000 2750 0    60   ~ 0
 VCCR
 Text Label 5250 3550 2    60   ~ 0
