File: kicad/bixi_pt/bixi_pt.kicad_pcb (KiCad board)
At the start: 2 copper layers, 47 x 21.6 mm, 5 parts, among them J1 Screw_Terminal_1x02, J2 CONN_01X03, J3 CONN_01X03

Commit message: v3 pcb's plotted, ready for fab
Parts:
- added burner-logo1: , logos:burner-logo-fs, F.Cu at (149.9, 82.5)
- added burner-logo2: , logos:burner-logo-fs, F.Cu at (178.4, 82.5)
- J2, J3: footprint Connectors_JST:JST_XH_B03B-XH-A_03x2.50mm_Straight -> custom:PAD_3X_OVAL_WS2812B
- moved J3 4.02 mm to (188.0, 87.6), turned to 180 degrees
- moved J2 1.80 mm to (147.3, 87.6), turned to 0 degrees
Routing:
- net /GND: track 0.00 -> 10.7 mm, vias 0 -> 2
- net /DATA: track 40.2 -> 44.3 mm

Commit message: first changes for v4 pcb's
Parts:
- added PWR_L: Jumper, Pin_Headers:Pin_Header_Straight_1x02_Pitch2.54mm, F.Cu at (152.9, 95.5)
- added PWR_R: Jumper, Pin_Headers:Pin_Header_Straight_1x02_Pitch2.54mm, F.Cu at (179.8, 95.5)
- moved REF** 2.40 mm to (147.3, 79.2)
- moved REF** 2.09 mm to (188.5, 79.2)
- moved burner-logo2 1.78 mm to (178.3, 80.8)
- moved burner-logo1 1.78 mm to (149.9, 80.8)
Connections:
- J2 pad 3: /VCC -> /VCCL
- J3 pad 1: /VCC -> /VCCR
Routing:
- net /GND: track 10.7 -> 0.00 mm, vias 2 -> 0
- net /VCCR: track 0.00 -> 8.06 mm
- net /VCCL: track 0.00 -> 8.06 mm
- net /DATA: track 44.3 -> 41.1 mm
- added copper zone on F.Cu, net /GND
- added copper zone on B.Cu, net /VCC
- removed copper zone on B.Cu, net /GND
- removed copper zone on F.Cu, net /VCC

Commit message: new power injection board is ready
Parts:
- removed J2, J3: CONN_01X03, custom:PAD_3X_OVAL_WS2812B
- removed PWR_L, PWR_R: Jumper, Pin_Headers:Pin_Header_Straight_1x02_Pitch2.54mm
- removed the REF** at (188.5, 79.2)
- removed the REF** at (147.3, 79.2)
- removed burner-logo1, burner-logo2: , logos:burner-logo-fs
- added L1: CONN_01X03, custom:3-wire-hole-with-relief, F.Cu at (118.5, 102.5)
- added PWR_L1: Jumper, Pin_Headers:Pin_Header_Straight_1x02_Pitch2.54mm, F.Cu at (117.0, 111.2)
- added PWR_R1: Jumper, Pin_Headers:Pin_Header_Straight_1x02_Pitch2.54mm, F.Cu at (141.5, 111.2)
- added R1: CONN_01X03, custom:3-wire-hole-with-relief, F.Cu at (142.2, 102.5)
- added REF**: MountingHole_3.5mm, Mounting_Holes:MountingHole_3.5mm, F.Cu at (130.3, 92.0)
- added REF**: MountingHole_3.5mm, Mounting_Holes:MountingHole_3.5mm, F.Cu at (130.3, 112.0)
- J1: footprint custom:HP_9500_Terminal_Connector -> custom:OSTYK42102030-2P-Terminal
- moved J1 38.7 mm to (130.4, 98.1)
Routing:
- net /VCC: track 0.00 -> 43.3 mm
- net /GND: track 0.00 -> 23.4 mm
- net /DATA: track 41.1 -> 21.8 mm
- net /VCCR: track 8.06 -> 9.46 mm
- net /VCCL: track 8.06 -> 9.34 mm
- removed copper zone on F.Cu, net /GND
- removed copper zone on B.Cu, net /VCC
Other:
- board size 47 x 21.6 mm -> 30.8 x 29 mm
- board text removed: "+"
- board text removed: "-"

Commit message: fixes to boards, node still in progress
Parts:
- added burner-logo: , logos:burner-logo-fs, F.Cu at (114.9, 87.6)
- added burner-logo: , logos:burner-logo-fs, F.Cu at (138.4, 87.6)
- renumbered REF** to S1, REF** to S2
Other:
- board size 30.8 x 29 mm -> 31 x 28 mm
- board text added: "+"
- board text added: "-"

Commit message: final v4 pcb's, sent to production
Parts:
- S1, S2: footprint Mounting_Holes:MountingHole_3.5mm -> Mounting_Holes:MountingHole_2.7mm_Pad
Changed lines of the file:
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@@
 (kicad_pcb (version 4) (host pcbnew 4.0.6)
   (general
-    (links 0)
+    (links 7)
     (no_connects 0)
-    (area 114.924999 87.924999 146.075001 116.075001)
+    (area 107.659286 83.871428 147.505 120.128571)
     (thickness 1.6)
     (drawings 24)
@@
     (add_net /VCCR)
   )
+  (module Mounting_Holes:MountingHole_2.7mm_Pad (layer F.Cu)
+    (at 130.3 112 90)
+    (descr "Mounting Hole 2.7mm")
+    (tags "mounting hole 2.7mm")
+    (fp_text reference S1 (at 0 -3.7 90) (layer F.SilkS)
+      (effects (font (size 1 1) (thickness 0.15)))
+    )
+    (fp_text value MountingHole_3.5mm (at 0 3.7 90) (layer F.Fab)
+      (effects (font (size 1 1) (thickness 0.15)))
+    )
+    (fp_circle (center 0 0) (end 2.7 0) (layer Cmts.User) (width 0.15))
+    (fp_circle (center 0 0) (end 2.95 0) (layer F.CrtYd) (width 0.05))
+    (pad 1 thru_hole circle (at 0 0 90) (size 5.4 5.4) (drill 2.7) (layers *.Cu *.Mask))
+  )
   (module logos:burner-logo-fs (layer F.Cu)
     (at 114.935 87.63)
@@
       (xy 5.94 10.65)) (layer F.SilkS) (width 0.01))
   )
-  (module Mounting_Holes:MountingHole_3.5mm (layer F.Cu)
-    (at 130.3 92 90)
-    (descr "Mounting Hole 3.5mm, no annular")
-    (tags "mounting hole 3.5mm no annular")
-    (fp_text reference S2 (at 5.64 -3.935 180) (layer F.SilkS)
-      (effects (font (size 1 1) (thickness 0.15)))
-    )
-    (fp_text value MountingHole_3.5mm (at 0 4.5 90) (layer F.Fab)
-      (effects (font (size 1 1) (thickness 0.15)))
-    )
-    (fp_circle (center 0 0) (end 3.5 0) (layer Cmts.User) (width 0.15))
-    (fp_circle (center 0 0) (end 3.75 0) (layer F.CrtYd) (width 0.05))
-    (pad 1 np_thru_hole circle (at 0 0 90) (size 3.5 3.5) (drill 3.5) (layers *.Cu *.Mask))
-  )
-  (module Mounting_Holes:MountingHole_3.5mm (layer F.Cu)
-    (at 130.3 112 90)
-    (descr "Mounting Hole 3.5mm, no annular")
-    (tags "mounting hole 3.5mm no annular")
-    (fp_text reference S1 (at -5.475 -3.3 180) (layer F.SilkS)
-      (effects (font (size 1 1) (thickness 0.15)))
-    )
-    (fp_text value MountingHole_3.5mm (at 0 4.5 90) (layer F.Fab)
-      (effects (font (size 1 1) (thickness 0.15)))
-    )
-    (fp_circle (center 0 0) (end 3.5 0) (layer Cmts.User) (width 0.15))
-    (fp_circle (center 0 0) (end 3.75 0) (layer F.CrtYd) (width 0.05))
-    (pad 1 np_thru_hole circle (at 0 0 90) (size 3.5 3.5) (drill 3.5) (layers *.Cu *.Mask))
-  )
   (module custom:OSTYK42102030-2P-Terminal (layer F.Cu)
     (at 130.4 98.1)
@@
       (xy 5.94 10.65)) (layer F.SilkS) (width 0.01))
   )
+  (module Mounting_Holes:MountingHole_2.7mm_Pad (layer F.Cu)
+    (at 130.3 92 90)
+    (descr "Mounting Hole 2.7mm")
+    (tags "mounting hole 2.7mm")
+    (fp_text reference S2 (at 0 -3.7 90) (layer F.SilkS)
+      (effects (font (size 1 1) (thickness 0.15)))
+    )
+    (fp_text value MountingHole_3.5mm (at 0 3.7 90) (layer F.Fab)
+      (effects (font (size 1 1) (thickness 0.15)))
+    )
+    (fp_circle (center 0 0) (end 2.7 0) (layer Cmts.User) (width 0.15))
+    (fp_circle (center 0 0) (end 2.95 0) (layer F.CrtYd) (width 0.05))
+    (pad 1 thru_hole circle (at 0 0 90) (size 5.4 5.4) (drill 2.7) (layers *.Cu *.Mask))
+  )
   (gr_line (start 115 113) (end 115 91) (angle 90) (layer Edge.Cuts) (width 0.15))
