File: kicad/bixi_node/bixi_node.kicad_pcb (KiCad board)
At the start: 2 copper layers, 48.3 x 16.5 mm, 8 parts, among them J1 RJ45, P1 CONN_01X03, U1 SP3485CN

Commit message: fixes to boards, node still in progress
Parts:
- removed burner-logo1, burner-logo2: , logos:burner-logo-fs
- added REF**: MountingHole_3.5mm_Pad, Mounting_Holes:MountingHole_3.5mm_Pad, F.Cu at (128.9, 85.1)
- added REF**: MountingHole_3.5mm_Pad, Mounting_Holes:MountingHole_3.5mm_Pad, F.Cu at (128.9, 96.5)
- P1: footprint custom:PAD_3X_OVAL_WS2812B -> custom:3-wire-hole-with-relief
- moved JP1 20.6 mm to (120.7, 86.4)
- moved P1 15.2 mm to (123.2, 91.2), turned to 0 degrees
- moved C1 8.26 mm to (108.0, 88.4)
- moved R1 8.25 mm to (108.0, 85.1)
- moved U1 6.99 mm to (109.2, 98.6)
Connections:
- P1 pad 1: VCC -> GND
- P1 pad 3: GND -> Net-(P1-Pad3)
Routing:
- net /DATA: track 26.7 -> 0.00 mm
- net /DATA_DIFF_A: track 25.7 -> 0.00 mm
- net /MODE: track 20.9 -> 0.00 mm
- net /DATA_DIFF_B: track 18.7 -> 0.00 mm
- net GND: track 5.35 -> 0.00 mm, vias 1 -> 0
- removed copper zone on B.Cu, net GND
- removed copper zone on F.Cu, net VCC
Other:
- board outline removed

Commit message: node work for keystone box
Parts:
- removed REF** (x2): MountingHole_3.5mm_Pad, Mounting_Holes:MountingHole_3.5mm_Pad
- added S1: MountingHole_2.7mm_Pad, Mounting_Holes:MountingHole_2.7mm_Pad, F.Cu at (60.8, 130.9)
- added S2: MountingHole_2.7mm_Pad, Mounting_Holes:MountingHole_2.7mm_Pad, F.Cu at (60.8, 142.9)
- moved R1 89.1 mm to (40.9, 143.8)
- moved J1 81.4 mm to (29.2, 137.2)
- moved JP1 80.3 mm to (53.6, 130.6)
- moved U1 79.3 mm to (42.2, 141.0)
- moved C1 79.2 mm to (40.9, 130.6)
- moved P1 77.4 mm to (60.7, 136.9)
Connections:
- P1 pad 3: Net-(P1-Pad3) -> VCC
Routing:
- added copper zone on B.Cu, net GND
- added copper zone on F.Cu, net VCC
Other:
- board outline added: 38.1 x 19.9 mm
- net class Default: trace_width 2 -> 0.4; via_dia 2 -> 0.4; via_drill 1 -> 0.3
- board text added: "100"
- board text added: "100nF"
- board text added: "5V"
- board text added: "DATA"
- board text added: "GND"
Changed lines of the file:
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@@
 (kicad_pcb (version 4) (host pcbnew 4.0.6)
   (general
-    (links 15)
-    (no_connects 15)
-    (area 88.370999 79.615 138.819286 102.656762)
+    (links 16)
+    (no_connects 8)
+    (area 20.32 124.46 75.751 149.860001)
     (thickness 1.6)
-    (drawings 2)
+    (drawings 11)
     (tracks 0)
     (zones 0)
     (modules 8)
-    (nets 12)
+    (nets 11)
   )
   (page A4)
@@
   )
   (setup
-    (last_trace_width 2)
+    (last_trace_width 0.4)
     (trace_clearance 0.2)
     (zone_clearance 0.508)
@@
     (segment_width 0.2)
     (edge_width 0.15)
-    (via_size 2)
-    (via_drill 1)
+    (via_size 0.4)
+    (via_drill 0.3)
     (via_min_size 0.4)
     (via_min_drill 0.3)
@@
     (mod_text_size 1 1)
     (mod_text_width 0.15)
-    (pad_size 1.524 1.524)
-    (pad_drill 0.762)
+    (pad_size 3.5 3.5)
+    (pad_drill 2.7)
     (pad_to_mask_clearance 0.2)
     (aux_axis_origin 0 0)
@@
   (net 9 "Net-(J1-Pad5)")
   (net 10 "Net-(J1-Pad6)")
-  (net 11 "Net-(P1-Pad3)")
   (net_class Default "This is the default net class."
     (clearance 0.2)
-    (trace_width 2)
-    (via_dia 2)
-    (via_drill 1)
+    (trace_width 0.4)
+    (via_dia 0.4)
+    (via_drill 0.3)
     (uvia_dia 0.3)
     (uvia_drill 0.1)
@@
     (add_net "Net-(J1-Pad5)")
     (add_net "Net-(J1-Pad6)")
-    (add_net "Net-(P1-Pad3)")
     (add_net VCC)
   )
+  (module Mounting_Holes:MountingHole_2.7mm_Pad locked (layer F.Cu)
+    (at 60.75 142.9255)
+    (descr "Mounting Hole 2.7mm")
+    (tags "mounting hole 2.7mm")
+    (fp_text reference S2 (at 10.116 -4.2415) (layer F.SilkS)
+      (effects (font (size 1 1) (thickness 0.15)))
+    )
+    (fp_text value MountingHole_2.7mm_Pad (at 20.276 5.6645) (layer F.Fab)
+      (effects (font (size 1 1) (thickness 0.15)))
+    )
+    (fp_circle (center 0 0) (end 2.7 0) (layer Cmts.User) (width 0.15))
+    (fp_circle (center 0 0) (end 2.95 0) (layer F.CrtYd) (width 0.05))
+    (pad 1 thru_hole circle (at 0 0) (size 3.5 3.5) (drill 2.7) (layers *.Cu *.Mask))
+  )
   (module Housings_DIP:DIP-8_W7.62mm (layer F.Cu)
-    (at 109.22 98.552 90)
+    (at 42.164 140.97 90)
     (descr "8-lead dip package, row spacing 7.62 mm (300 mils)")
     (tags "dil dip 2.54 300")
@@
   )
   (module Connectors:RJ45_8 (layer F.Cu)
-    (at 96.52 91.44 270)
+    (at 29.21 137.16 270)
     (tags RJ45)
-    (fp_text reference J1 (at 0.254 4.826 270) (layer F.SilkS)
+    (fp_text reference J1 (at 0 -3.048 270) (layer F.SilkS)
       (effects (font (size 1 1) (thickness 0.15)))
     )
@@
   )
   (module Resistors_THT:Resistor_Horizontal_RM7mm (layer F.Cu)
-    (at 107.95 85.09)
+    (at 40.894 143.764)
     (descr "Resistor, Axial,  RM 7.62mm, 1/3W,")
     (tags "Resistor Axial RM 7.62mm 1/3W R3")
-    (fp_text reference R1 (at 4 2.5) (layer F.SilkS)
+    (fp_text reference R1 (at 3.81 2.286) (layer F.SilkS)
       (effects (font (size 1 1) (thickness 0.15)))
     )
@@
   )
   (module custom:jumper_3_pin_fixed (layer F.Cu)
-    (at 120.65 86.36)
-    (fp_text reference JP1 (at -5.08 -1.27) (layer F.SilkS)
-      (effects (font (size 1 1) (thickness 0.15)))
-    )
-    (fp_text value Jumper_NC_Dual (at 0 -0.5) (layer F.Fab)
+    (at 53.594 130.556)
+    (fp_text reference JP1 (at 3.048 -22.606) (layer F.SilkS)
+      (effects (font (size 1 1) (thickness 0.15)))
+    )
+    (fp_text value Jumper_NC_Dual (at 2.794 -19.812) (layer F.Fab)
       (effects (font (size 1 1) (thickness 0.15)))
     )
@@
   )
   (module Capacitors_THT:C_Axial_L3.8mm_D2.6mm_P7.50mm_Horizontal (layer F.Cu)
-    (at 107.95 88.392)
+    (at 40.894 130.556)
     (descr "C, Axial series, Axial, Horizontal, pin pitch=7.5mm, , length*diameter=3.8*2.6mm^2, http://www.vishay.com/docs/45231/arseries.pdf")
     (tags "C Axial series Axial Horizontal pin pitch 7.5mm  length 3.8mm diameter 2.6mm")
@@
   )
   (module custom:3-wire-hole-with-relief (layer F.Cu)
-    (at 123.19 91.186)
+    (at 60.706 136.906)
     (fp_text reference P1 (at 0.254 -4.572) (layer F.SilkS)
       (effects (font (size 1 1) (thickness 0.15)))
     )
-    (fp_text value CONN_01X03 (at -0.27 -0.5) (layer F.Fab)
+    (fp_text value CONN_01X03 (at 23.368 1.27) (layer F.Fab)
       (effects (font (size 1 1) (thickness 0.15)))
     )
@@
       (net 4 /DATA))
     (pad 3 thru_hole circle (at -1.81 2.54) (size 1.778 1.778) (drill 1.016) (layers *.Cu *.Mask)
-      (net 11 "Net-(P1-Pad3)"))
+      (net 1 VCC))
     (pad "" np_thru_hole circle (at 1 -2.54) (size 2.286 2.286) (drill 2.032) (layers *.Cu *.Mask))
     (pad "" np_thru_hole circle (at 1 0) (size 2.286 2.286) (drill 2.032) (layers *.Cu *.Mask))
     (pad "" np_thru_hole circle (at 1 2.54) (size 2.286 2.286) (drill 2.032) (layers *.Cu *.Mask))
   )
-  (module Mounting_Holes:MountingHole_3.5mm_Pad (layer F.Cu)
-    (at 128.905 85.09)
-    (descr "Mounting Hole 3.5mm")
-    (tags "mounting hole 3.5mm")
-    (fp_text reference REF** (at 0 -4.5) (layer F.SilkS)
-      (effects (font (size 1 1) (thickness 0.15)))
-    )
-    (fp_text value MountingHole_3.5mm_Pad (at 0 4.5) (layer F.Fab)
-      (effects (font (size 1 1) (thickness 0.15)))
-    )
-    (fp_circle (center 0 0) (end 3.5 0) (layer Cmts.User) (width 0.15))
-    (fp_circle (center 0 0) (end 3.75 0) (layer F.CrtYd) (width 0.05))
-    (pad 1 thru_hole circle (at 0 0) (size 7 7) (drill 3.5) (layers *.Cu *.Mask))
-  )
-  (module Mounting_Holes:MountingHole_3.5mm_Pad (layer F.Cu)
-    (at 128.905 96.52)
-    (descr "Mounting Hole 3.5mm")
-    (tags "mounting hole 3.5mm")
-    (fp_text reference REF** (at 0 -4.5) (layer F.SilkS)
-      (effects (font (size 1 1) (thickness 0.15)))
-    )
-    (fp_text value MountingHole_3.5mm_Pad (at 0 4.5) (layer F.Fab)
-      (effects (font (size 1 1) (thickness 0.15)))
-    )
-    (fp_circle (center 0 0) (end 3.5 0) (layer Cmts.User) (width 0.15))
-    (fp_circle (center 0 0) (end 3.75 0) (layer F.CrtYd) (width 0.05))
-    (pad 1 thru_hole circle (at 0 0) (size 7 7) (drill 3.5) (layers *.Cu *.Mask))
-  )
-  (gr_text RX (at 121.92 84.836) (layer F.SilkS)
+  (module Mounting_Holes:MountingHole_2.7mm_Pad locked (layer F.Cu)
+    (at 60.75 130.95)
+    (descr "Mounting Hole 2.7mm")
+    (tags "mounting hole 2.7mm")
+    (fp_text reference S1 (at 10.878 -4.204) (layer F.SilkS)
+      (effects (font (size 1 1) (thickness 0.15)))
+    )
+    (fp_text value MountingHole_2.7mm_Pad (at 22.562 -1.41) (layer F.Fab)
+      (effects (font (size 1 1) (thickness 0.15)))
+    )
+    (fp_circle (center 0 0) (end 2.7 0) (layer Cmts.User) (width 0.15))
+    (fp_circle (center 0 0) (end 2.95 0) (layer F.CrtYd) (width 0.05))
+    (pad 1 thru_hole circle (at 0 0) (size 3.5 3.5) (drill 2.7) (layers *.Cu *.Mask))
+  )
+  (gr_text 5V (at 56.388 139.446) (layer F.SilkS)
+    (effects (font (size 1 1) (thickness 0.25)))
+  )
+  (gr_text DATA (at 55.626 136.906) (layer F.SilkS)
+    (effects (font (size 1 1) (thickness 0.25)))
+  )
+  (gr_text GND (at 55.88 134.366) (layer F.SilkS)
+    (effects (font (size 1 1) (thickness 0.25)))
+  )
+  (gr_text 100 (at 44.704 143.764) (layer F.SilkS)
+    (effects (font (size 1.5 1.5) (thickness 0.3)))
+  )
+  (gr_text 100nF (at 44.704 130.556) (layer F.SilkS)
+    (effects (font (size 1.5 0.75) (thickness 0.1875)))
+  )
+  (gr_line (start 25.4 146.8755) (end 63.5 146.8755) (angle 90) (layer Edge.Cuts) (width 0.15))
+  (gr_line (start 63.5 127) (end 63.5 146.8755) (angle 90) (layer Edge.Cuts) (width 0.15))
+  (gr_line (start 25.4 127) (end 25.4 146.8755) (angle 90) (layer Edge.Cuts) (width 0.15))
+  (gr_line (start 25.4 127) (end 63.5 127) (angle 90) (layer Edge.Cuts) (width 0.15))
+  (gr_text RX (at 54.864 129.032) (layer F.SilkS)
     (effects (font (size 1 1) (thickness 0.15)))
   )
-  (gr_text TX (at 119.38 84.836) (layer F.SilkS)
+  (gr_text TX (at 52.324 129.032) (layer F.SilkS)
     (effects (font (size 1 1) (thickness 0.15)))
   )
+  (zone (net 1) (net_name VCC) (layer F.Cu) (hatch edge 0.508)
+    (connect_pads (clearance 0.508))
+    (min_thickness 0.254)
+    (fill yes (arc_segments 16) (thermal_gap 1) (thermal_bridge_width 1))
+    (polygon
+      (pts
+        (xy 66.04 149.86) (xy 20.32 149.86) (xy 20.32 124.46) (xy 66.04 124.46)
+      )
+    )
+  )
+  (zone (net 2) (net_name GND) (layer B.Cu) (hatch edge 0.508)
+    (connect_pads (clearance 0.508))
+    (min_thickness 0.254)
+    (fill yes (arc_segments 16) (thermal_gap 1) (thermal_bridge_width 1))
+    (polygon
+      (pts
+        (xy 66.04 149.86) (xy 20.32 149.86) (xy 20.32 124.46) (xy 66.04 124.46)
+      )
+    )
+  )
 )

Commit message: final v4 pcb's, sent to production
Connections:
- net /MODE renamed /MD
Routing:
- net /DATA_DIFF_A: track 0.00 -> 24.3 mm
- net /DATA_DIFF_B: track 0.00 -> 20.0 mm
- net /DATA: track 0.00 -> 19.6 mm
- net /MD: track 0.00 -> 15.6 mm
Changed lines of the file:
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@@
   (general
     (links 16)
-    (no_connects 8)
-    (area 20.32 124.46 75.751 149.860001)
+    (no_connects 0)
+    (area 20.32 106.975 93.226286 149.860001)
     (thickness 1.6)
     (drawings 11)
-    (tracks 0)
+    (tracks 27)
     (zones 0)
     (modules 8)
@@
   (net 5 /DATA_DIFF_A)
   (net 6 /DATA_DIFF_B)
-  (net 7 /MODE)
-  (net 8 "Net-(J1-Pad3)")
-  (net 9 "Net-(J1-Pad5)")
-  (net 10 "Net-(J1-Pad6)")
+  (net 7 "Net-(J1-Pad3)")
+  (net 8 "Net-(J1-Pad5)")
+  (net 9 "Net-(J1-Pad6)")
+  (net 10 /MD)
   (net_class Default "This is the default net class."
     (clearance 0.2)
@@
     (add_net /DATA_DIFF_A)
     (add_net /DATA_DIFF_B)
-    (add_net /MODE)
+    (add_net /MD)
     (add_net GND)
     (add_net "Net-(J1-Pad3)")
@@
   )
   (module Mounting_Holes:MountingHole_2.7mm_Pad locked (layer F.Cu)
-    (at 60.75 142.9255)
+    (at 60.75 142.926)
     (descr "Mounting Hole 2.7mm")
     (tags "mounting hole 2.7mm")
@@
       (net 4 /DATA))
     (pad 2 thru_hole oval (at 0 2.54 90) (size 1.6 1.6) (drill 0.8) (layers *.Cu *.Mask)
-      (net 7 /MODE))
+      (net 10 /MD))
     (pad 3 thru_hole oval (at 0 5.08 90) (size 1.6 1.6) (drill 0.8) (layers *.Cu *.Mask)
-      (net 7 /MODE))
+      (net 10 /MD))
     (pad 4 thru_hole oval (at 0 7.62 90) (size 1.6 1.6) (drill 0.8) (layers *.Cu *.Mask)
       (net 4 /DATA))
@@
       (net 6 /DATA_DIFF_B))
     (pad 3 thru_hole circle (at -1.905 -6.35 270) (size 1.50114 1.50114) (drill 0.89916) (layers *.Cu *.Mask)
-      (net 8 "Net-(J1-Pad3)"))
+      (net 7 "Net-(J1-Pad3)"))
     (pad 4 thru_hole circle (at -0.635 -8.89 270) (size 1.50114 1.50114) (drill 0.89916) (layers *.Cu *.Mask)
       (net 3 "Net-(J1-Pad4)"))
     (pad 5 thru_hole circle (at 0.635 -6.35 270) (size 1.50114 1.50114) (drill 0.89916) (layers *.Cu *.Mask)
-      (net 9 "Net-(J1-Pad5)"))
+      (net 8 "Net-(J1-Pad5)"))
     (pad 6 thru_hole circle (at 1.905 -8.89 270) (size 1.50114 1.50114) (drill 0.89916) (layers *.Cu *.Mask)
-      (net 10 "Net-(J1-Pad6)"))
+      (net 9 "Net-(J1-Pad6)"))
     (pad 7 thru_hole circle (at 3.175 -6.35 270) (size 1.50114 1.50114) (drill 0.89916) (layers *.Cu *.Mask)
       (net 2 GND))
@@
       (net 1 VCC))
     (pad 2 thru_hole circle (at 0 0) (size 1.524 1.524) (drill 0.762) (layers *.Cu *.Mask)
-      (net 7 /MODE))
+      (net 10 /MD))
     (pad 3 thru_hole circle (at 2.54 0) (size 1.524 1.524) (drill 0.762) (layers *.Cu *.Mask)
       (net 2 GND))
@@
       (effects (font (size 1 1) (thickness 0.15)))
     )
-    (fp_text value C (at 3.75 2.36) (layer F.Fab)
+    (fp_text value C (at 11.176 -4.826) (layer F.Fab)
       (effects (font (size 1 1) (thickness 0.15)))
     )
@@
     (effects (font (size 1 1) (thickness 0.15)))
   )
+  (segment (start 42.164 140.97) (end 42.164 141.224) (width 0.4) (layer F.Cu) (net 4))
+  (segment (start 42.164 141.224) (end 43.18 142.24) (width 0.4) (layer F.Cu) (net 4))
+  (segment (start 43.18 142.24) (end 48.514 142.24) (width 0.4) (layer F.Cu) (net 4))
+  (segment (start 48.514 142.24) (end 49.784 140.97) (width 0.4) (layer F.Cu) (net 4))
+  (segment (start 49.784 140.97) (end 54.832 140.97) (width 0.4) (layer F.Cu) (net 4))
+  (segment (start 54.832 140.97) (end 58.896 136.906) (width 0.4) (layer F.Cu) (net 4))
+  (segment (start 47.244 133.35) (end 47.244 133.604) (width 0.4) (layer B.Cu) (net 5))
+  (segment (start 47.244 133.604) (end 45.974 134.874) (width 0.4) (layer B.Cu) (net 5))
+  (segment (start 38.989 132.715) (end 35.56 132.715) (width 0.4) (layer B.Cu) (net 5))
+  (segment (start 41.148 134.874) (end 38.989 132.715) (width 0.4) (layer B.Cu) (net 5))
+  (segment (start 45.974 134.874) (end 41.148 134.874) (width 0.4) (layer B.Cu) (net 5))
+  (segment (start 48.514 143.764) (end 48.514 135.636) (width 0.4) (layer B.Cu) (net 5))
+  (segment (start 47.244 134.366) (end 47.244 133.35) (width 0.4) (layer B.Cu) (net 5))
+  (segment (start 48.514 135.636) (end 47.244 134.366) (width 0.4) (layer B.Cu) (net 5))
+  (segment (start 40.894 143.764) (end 40.894 142.24) (width 0.4) (layer B.Cu) (net 6))
+  (segment (start 39.878 135.763) (end 38.1 133.985) (width 0.4) (layer B.Cu) (net 6))
+  (segment (start 39.878 141.224) (end 39.878 135.763) (width 0.4) (layer B.Cu) (net 6))
+  (segment (start 40.894 142.24) (end 39.878 141.224) (width 0.4) (layer B.Cu) (net 6))
+  (segment (start 38.1 133.985) (end 40.005 133.985) (width 0.4) (layer F.Cu) (net 6))
+  (segment (start 44.704 134.366) (end 44.704 133.35) (width 0.4) (layer F.Cu) (net 6))
+  (segment (start 43.18 135.89) (end 44.704 134.366) (width 0.4) (layer F.Cu) (net 6))
+  (segment (start 41.91 135.89) (end 43.18 135.89) (width 0.4) (layer F.Cu) (net 6))
+  (segment (start 40.005 133.985) (end 41.91 135.89) (width 0.4) (layer F.Cu) (net 6))
+  (segment (start 47.244 140.97) (end 47.244 138.938) (width 1) (layer F.Cu) (net 10))
+  (segment (start 53.594 132.588) (end 53.594 130.556) (width 1) (layer F.Cu) (net 10))
+  (segment (start 47.244 138.938) (end 53.594 132.588) (width 1) (layer F.Cu) (net 10))
+  (segment (start 44.704 140.97) (end 47.244 140.97) (width 1) (layer F.Cu) (net 10))
   (zone (net 1) (net_name VCC) (layer F.Cu) (hatch edge 0.508)
     (connect_pads (clearance 0.508))
