File: kicad/bixi_node/bixi_node.sch (KiCad schematic (older format))
At the start: 6 parts, among them J1 RJ45, P1 CONN_01X03, U1 SP3485CN

Commit message: fixes to boards, node still in progress
Parts:
- P1: footprint custom:PAD_3X_OVAL_WS2812B -> custom:3-wire-hole-with-relief
Connections:
- net GND: now also P1.1 (P1); no longer P1.3 (P3)
- net VCC: no longer P1.1 (P1)
Other:
- moved on the sheet: P1
Changed lines of the file:
@@
 L VCC #PWR07
 U 1 1 58D6B5B6
-P 8050 3200
-F 0 "#PWR07" H 8050 3050 50  0001 C CNN
-F 1 "VCC" H 8050 3350 50  0000 C CNN
-F 2 "" H 8050 3200 50  0000 C CNN
-F 3 "" H 8050 3200 50  0000 C CNN
-	1    8050 3200
+P 8400 3850
+F 0 "#PWR07" H 8400 3700 50  0001 C CNN
+F 1 "VCC" H 8400 4000 50  0000 C CNN
+F 2 "" H 8400 3850 50  0000 C CNN
+F 3 "" H 8400 3850 50  0000 C CNN
+	1    8400 3850
 	1    0    0    -1
 $EndComp
@@
 L GND #PWR08
 U 1 1 58D6B5DA
-P 8050 3400
-F 0 "#PWR08" H 8050 3150 50  0001 C CNN
-F 1 "GND" H 8050 3250 50  0000 C CNN
-F 2 "" H 8050 3400 50  0000 C CNN
-F 3 "" H 8050 3400 50  0000 C CNN
-	1    8050 3400
+P 8400 4150
+F 0 "#PWR08" H 8400 3900 50  0001 C CNN
+F 1 "GND" H 8400 4000 50  0000 C CNN
+F 2 "" H 8400 4150 50  0000 C CNN
+F 3 "" H 8400 4150 50  0000 C CNN
+	1    8400 4150
 	1    0    0    -1
 $EndComp
@@
 L CONN_01X03 P1
 U 1 1 58D6C384
-P 8250 3300
-F 0 "P1" H 8250 3500 50  0000 C CNN
-F 1 "CONN_01X03" V 8350 3300 50  0000 C CNN
-F 2 "custom:PAD_3X_OVAL_WS2812B" H 8250 3300 50  0001 C CNN
-F 3 "" H 8250 3300 50  0000 C CNN
-	1    8250 3300
-	1    0    0    -1
+P 8200 4050
+F 0 "P1" H 8200 4250 50  0000 C CNN
+F 1 "CONN_01X03" V 8300 4050 50  0000 C CNN
+F 2 "custom:3-wire-hole-with-relief" H 8200 4050 50  0001 C CNN
+F 3 "" H 8200 4050 50  0000 C CNN
+	1    8200 4050
+	-1   0    0    1
 $EndComp
 $Comp
@@
 	0    1    1    0
 $EndComp
-Text Label 8050 3300 2    60   ~ 0
+Text Label 8400 4050 0    60   ~ 0
 DATA
 $Comp

Commit message: node work for keystone box
Connections:
- net VCC: now also P1.3 (P3)
Changed lines of the file:
@@
 L VCC #PWR07
 U 1 1 58D6B5B6
-P 8400 3850
-F 0 "#PWR07" H 8400 3700 50  0001 C CNN
-F 1 "VCC" H 8400 4000 50  0000 C CNN
-F 2 "" H 8400 3850 50  0000 C CNN
-F 3 "" H 8400 3850 50  0000 C CNN
-	1    8400 3850
+P 8400 3950
+F 0 "#PWR07" H 8400 3800 50  0001 C CNN
+F 1 "VCC" H 8400 4100 50  0000 C CNN
+F 2 "" H 8400 3950 50  0000 C CNN
+F 3 "" H 8400 3950 50  0000 C CNN
+	1    8400 3950
 	1    0    0    -1
 $EndComp

Commit message: final v4 pcb's, sent to production
Connections:
- net MODE renamed MD
Changed lines of the file:
@@
 DATA_DIFF_B
 Text Label 5400 3200 2    60   ~ 0
-MODE
+MD
 Text Label 5400 3400 2    60   ~ 0
-MODE
+MD
 Text Label 6300 4800 2    60   ~ 0
-MODE
+MD
 $EndSCHEMATC
